File: JF-PimpleClock.kicad_sch (KiCad schematic)
At the start: 58 parts, among them J1 Conn_01x06_Female, J2 Conn_01x02, J3 Conn_01x02, J4 USB_B_Micro, Q1 Q_PMOS_DSG, SW1 SW_Push, SW2 SW_Push, SW3 SW_Push, SW4 SW_Push, U1 ATmega328-P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

Commit message: revisions for pcb layout, new cheaper parts selected, this went out into a test production
Parts:
- D1: footprint Diode_SMD:D_0402_1005Metric -> Diode_SMD:D_SMA
- Dh1, Dh2, Dh3, Dh4, Dm1, Dm2, Dm3, Dm4, Dm5, Dm6: footprint LED_SMD:LED_WS2812B-2020_PLCC4_2.0x2.0mm -> LED_THT:LED_D5.0mm-4_RGB
- J2: footprint Connector_JST:JST_EH_S2B-EH_1x02_P2.50mm_Horizontal -> Connector_JST:JST_PH_S2B-PH-K_1x02_P2.00mm_Horizontal
- U1: footprint Package_DIP:DIP-28_W7.62mm -> Package_QFP:TQFP-32_7x7mm_P0.8mm
Changed lines of the file:
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@@
     (property "Reference" "Dm2" (id 0) (at 165.1 94.7293 0))
     (property "Value" "NeoPixel_THT" (id 1) (at 165.1 97.2693 0))
-    (property "Footprint" "LED_SMD:LED_WS2812B-2020_PLCC4_2.0x2.0mm" (id 2) (at 153.67 106.68 0)
+    (property "Footprint" "LED_THT:LED_D5.0mm-4_RGB" (id 2) (at 153.67 106.68 0)
       (effects (font (size 1.27 1.27)) (justify left top) hide)
     )
@@
     (property "Reference" "U1" (id 0) (at 21.59 20.32 0))
     (property "Value" "ATmega328-P" (id 1) (at 41.91 93.98 0))
-    (property "Footprint" "Package_DIP:DIP-28_W7.62mm" (id 2) (at 33.02 57.15 0)
+    (property "Footprint" "Package_QFP:TQFP-32_7x7mm_P0.8mm" (id 2) (at 33.02 57.15 0)
       (effects (font (size 1.27 1.27) italic) hide)
     )
@@
     (property "Reference" "Dm1" (id 0) (at 137.16 94.7293 0))
     (property "Value" "NeoPixel_THT" (id 1) (at 137.16 97.2693 0))
-    (property "Footprint" "LED_SMD:LED_WS2812B-2020_PLCC4_2.0x2.0mm" (id 2) (at 125.73 106.68 0)
+    (property "Footprint" "LED_THT:LED_D5.0mm-4_RGB" (id 2) (at 125.73 106.68 0)
       (effects (font (size 1.27 1.27)) (justify left top) hide)
     )
@@
     (property "Reference" "Dh3" (id 0) (at 248.92 70.5993 0))
     (property "Value" "NeoPixel_THT" (id 1) (at 248.92 73.1393 0))
-    (property "Footprint" "LED_SMD:LED_WS2812B-2020_PLCC4_2.0x2.0mm" (id 2) (at 237.49 82.55 0)
+    (property "Footprint" "LED_THT:LED_D5.0mm-4_RGB" (id 2) (at 237.49 82.55 0)
       (effects (font (size 1.27 1.27)) (justify left top) hide)
     )
@@
       (effects (font (size 0.5 0.5)) (justify left))
     )
-    (property "Footprint" "Connector_JST:JST_EH_S2B-EH_1x02_P2.50mm_Horizontal" (id 2) (at 102.87 163.83 0)
+    (property "Footprint" "Connector_JST:JST_PH_S2B-PH-K_1x02_P2.00mm_Horizontal" (id 2) (at 102.87 163.83 0)
       (effects (font (size 1.27 1.27)) hide)
     )
@@
     (property "Reference" "Dh1" (id 0) (at 193.04 70.5993 0))
     (property "Value" "NeoPixel_THT" (id 1) (at 193.04 73.1393 0))
-    (property "Footprint" "LED_SMD:LED_WS2812B-2020_PLCC4_2.0x2.0mm" (id 2) (at 181.61 82.55 0)
+    (property "Footprint" "LED_THT:LED_D5.0mm-4_RGB" (id 2) (at 181.61 82.55 0)
       (effects (font (size 1.27 1.27)) (justify left top) hide)
     )
@@
     (property "Reference" "D1" (id 0) (at 124.7775 135.89 0))
     (property "Value" "D_Schottky" (id 1) (at 124.7775 138.43 0))
-    (property "Footprint" "Diode_SMD:D_0402_1005Metric" (id 2) (at 124.46 142.24 0)
+    (property "Footprint" "Diode_SMD:D_SMA" (id 2) (at 124.46 142.24 0)
       (effects (font (size 1.27 1.27)) hide)
     )
@@
     (property "Reference" "Dh4" (id 0) (at 275.59 70.5993 0))
     (property "Value" "NeoPixel_THT" (id 1) (at 275.59 73.1393 0))
-    (property "Footprint" "LED_SMD:LED_WS2812B-2020_PLCC4_2.0x2.0mm" (id 2) (at 264.16 82.55 0)
+    (property "Footprint" "LED_THT:LED_D5.0mm-4_RGB" (id 2) (at 264.16 82.55 0)
       (effects (font (size 1.27 1.27)) (justify left top) hide)
     )
@@
     (property "Reference" "Dm5" (id 0) (at 248.92 94.7293 0))
     (property "Value" "NeoPixel_THT" (id 1) (at 248.92 97.2693 0))
-    (property "Footprint" "LED_SMD:LED_WS2812B-2020_PLCC4_2.0x2.0mm" (id 2) (at 237.49 106.68 0)
+    (property "Footprint" "LED_THT:LED_D5.0mm-4_RGB" (id 2) (at 237.49 106.68 0)
       (effects (font (size 1.27 1.27)) (justify left top) hide)
     )
@@
     (property "Reference" "Dh2" (id 0) (at 220.98 70.5993 0))
     (property "Value" "NeoPixel_THT" (id 1) (at 220.98 73.1393 0))
-    (property "Footprint" "LED_SMD:LED_WS2812B-2020_PLCC4_2.0x2.0mm" (id 2) (at 209.55 82.55 0)
+    (property "Footprint" "LED_THT:LED_D5.0mm-4_RGB" (id 2) (at 209.55 82.55 0)
       (effects (font (size 1.27 1.27)) (justify left top) hide)
     )
@@
     (property "Reference" "Dm6" (id 0) (at 275.59 94.7293 0))
     (property "Value" "NeoPixel_THT" (id 1) (at 275.59 97.2693 0))
-    (property "Footprint" "LED_SMD:LED_WS2812B-2020_PLCC4_2.0x2.0mm" (id 2) (at 264.16 106.68 0)
+    (property "Footprint" "LED_THT:LED_D5.0mm-4_RGB" (id 2) (at 264.16 106.68 0)
       (effects (font (size 1.27 1.27)) (justify left top) hide)
     )
@@
     (property "Reference" "Dm3" (id 0) (at 193.04 94.7293 0))
     (property "Value" "NeoPixel_THT" (id 1) (at 193.04 97.2693 0))
-    (property "Footprint" "LED_SMD:LED_WS2812B-2020_PLCC4_2.0x2.0mm" (id 2) (at 181.61 106.68 0)
+    (property "Footprint" "LED_THT:LED_D5.0mm-4_RGB" (id 2) (at 181.61 106.68 0)
       (effects (font (size 1.27 1.27)) (justify left top) hide)
     )
@@
     (property "Reference" "Dm4" (id 0) (at 219.71 94.7293 0))
     (property "Value" "NeoPixel_THT" (id 1) (at 219.71 97.2693 0))
-    (property "Footprint" "LED_SMD:LED_WS2812B-2020_PLCC4_2.0x2.0mm" (id 2) (at 208.28 106.68 0)
+    (property "Footprint" "LED_THT:LED_D5.0mm-4_RGB" (id 2) (at 208.28 106.68 0)
       (effects (font (size 1.27 1.27)) (justify left top) hide)
     )
@@
     )
     (path "/8544b940-a52f-40fd-ae95-c83f0245f4b3"
-      (reference "D1") (unit 1) (value "D_Schottky") (footprint "Diode_SMD:D_0402_1005Metric")
+      (reference "D1") (unit 1) (value "D_Schottky") (footprint "Diode_SMD:D_SMA")
     )
     (path "/8472f604-424d-47af-a6dd-04d2a273b203"
-      (reference "Dh1") (unit 1) (value "NeoPixel_THT") (footprint "LED_SMD:LED_WS2812B-2020_PLCC4_2.0x2.0mm")
+      (reference "Dh1") (unit 1) (value "NeoPixel_THT") (footprint "LED_THT:LED_D5.0mm-4_RGB")
     )
     (path "/a61cf4c7-6f05-411f-a395-591c2c8c09ba"
-      (reference "Dh2") (unit 1) (value "NeoPixel_THT") (footprint "LED_SMD:LED_WS2812B-2020_PLCC4_2.0x2.0mm")
+      (reference "Dh2") (unit 1) (value "NeoPixel_THT") (footprint "LED_THT:LED_D5.0mm-4_RGB")
     )
     (path "/3d48d436-748f-4067-ba9d-2e776ee168a4"
-      (reference "Dh3") (unit 1) (value "NeoPixel_THT") (footprint "LED_SMD:LED_WS2812B-2020_PLCC4_2.0x2.0mm")
+      (reference "Dh3") (unit 1) (value "NeoPixel_THT") (footprint "LED_THT:LED_D5.0mm-4_RGB")
     )
     (path "/8552c7ad-a3b3-458a-99c8-abf7182d505b"
-      (reference "Dh4") (unit 1) (value "NeoPixel_THT") (footprint "LED_SMD:LED_WS2812B-2020_PLCC4_2.0x2.0mm")
+      (reference "Dh4") (unit 1) (value "NeoPixel_THT") (footprint "LED_THT:LED_D5.0mm-4_RGB")
     )
     (path "/39c0f5f7-c608-4a37-b98c-6420f0414324"
-      (reference "Dm1") (unit 1) (value "NeoPixel_THT") (footprint "LED_SMD:LED_WS2812B-2020_PLCC4_2.0x2.0mm")
+      (reference "Dm1") (unit 1) (value "NeoPixel_THT") (footprint "LED_THT:LED_D5.0mm-4_RGB")
     )
     (path "/1fdc9459-7f70-4323-8267-176e7549812c"
-      (reference "Dm2") (unit 1) (value "NeoPixel_THT") (footprint "LED_SMD:LED_WS2812B-2020_PLCC4_2.0x2.0mm")
+      (reference "Dm2") (unit 1) (value "NeoPixel_THT") (footprint "LED_THT:LED_D5.0mm-4_RGB")
     )
     (path "/d346081a-9c81-4ab6-957d-44af484be7b9"
-      (reference "Dm3") (unit 1) (value "NeoPixel_THT") (footprint "LED_SMD:LED_WS2812B-2020_PLCC4_2.0x2.0mm")
+      (reference "Dm3") (unit 1) (value "NeoPixel_THT") (footprint "LED_THT:LED_D5.0mm-4_RGB")
     )
     (path "/ee5f3bf7-0551-48c6-96a4-8b5133791144"
-      (reference "Dm4") (unit 1) (value "NeoPixel_THT") (footprint "LED_SMD:LED_WS2812B-2020_PLCC4_2.0x2.0mm")
+      (reference "Dm4") (unit 1) (value "NeoPixel_THT") (footprint "LED_THT:LED_D5.0mm-4_RGB")
     )
     (path "/90e3aeec-95cd-46a4-a076-2bf052844e47"
-      (reference "Dm5") (unit 1) (value "NeoPixel_THT") (footprint "LED_SMD:LED_WS2812B-2020_PLCC4_2.0x2.0mm")
+      (reference "Dm5") (unit 1) (value "NeoPixel_THT") (footprint "LED_THT:LED_D5.0mm-4_RGB")
     )
     (path "/b86083e9-9c48-4bcc-afce-f48b7c514ff4"
-      (reference "Dm6") (unit 1) (value "NeoPixel_THT") (footprint "LED_SMD:LED_WS2812B-2020_PLCC4_2.0x2.0mm")
+      (reference "Dm6") (unit 1) (value "NeoPixel_THT") (footprint "LED_THT:LED_D5.0mm-4_RGB")
     )
     (path "/89c7713b-1f3b-410b-b111-d1fd07f9eace"
@@
     )
     (path "/42ef20e1-61f8-40f2-a140-a2c91fececca"
-      (reference "J2") (unit 1) (value "Conn_01x02") (footprint "Connector_JST:JST_EH_S2B-EH_1x02_P2.50mm_Horizontal")
+      (reference "J2") (unit 1) (value "Conn_01x02") (footprint "Connector_JST:JST_PH_S2B-PH-K_1x02_P2.00mm_Horizontal")
     )
     (path "/014bcc5a-4d68-467a-b14f-a84ab8b56487"
@@
     )
     (path "/28ffd0b3-acb5-4327-bccd-b76ede86bb21"
-      (reference "U1") (unit 1) (value "ATmega328-P") (footprint "Package_DIP:DIP-28_W7.62mm")
+      (reference "U1") (unit 1) (value "ATmega328-P") (footprint "Package_QFP:TQFP-32_7x7mm_P0.8mm")
     )
     (path "/d860bdbb-6e93-4324-9516-c7eec4702ee5"

Commit message: small circuit tweak for fixing missing vcc/avcc ref for bootloader
Parts:
- added C19: 100nF, Capacitor_SMD:C_0805_2012Metric, symbol Device:C
Connections:
- net 5v: now also U1.20 (AVCC), C19.2
- net GND: now also C19.1
- no-connect marks 24 -> 23
Changed lines of the file:
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@@
     (company "DCR")
   )
+  (junction (at 33.02 17.78) (diameter 0) (color 0 0 0 0)
+  )
   (junction (at 123.19 184.15) (diameter 0) (color 0 0 0 0)
   )
@@
   )
   (junction (at 180.34 107.95) (diameter 0) (color 0 0 0 0)
+  )
+  (junction (at 35.56 17.78) (diameter 0) (color 0 0 0 0)
   )
   (junction (at 236.22 109.22) (diameter 0) (color 0 0 0 0)
@@
   (no_connect (at 101.6 116.84))
   (no_connect (at 48.26 36.83))
-  (no_connect (at 35.56 19.05))
   (no_connect (at 219.71 135.89))
   (no_connect (at 48.26 54.61))
@@
     (stroke (width 0) (type default) (color 0 0 0 0))
   )
+  (wire (pts (xy 63.5 26.67) (xy 63.5 27.94))
+    (stroke (width 0) (type default) (color 0 0 0 0))
+  )
   (wire (pts (xy 179.07 36.83) (xy 179.07 39.37))
     (stroke (width 0) (type default) (color 0 0 0 0))
@@
     (stroke (width 0) (type default) (color 0 0 0 0))
   )
+  (wire (pts (xy 33.02 17.78) (xy 35.56 17.78))
+    (stroke (width 0) (type default) (color 0 0 0 0))
+  )
   (wire (pts (xy 171.45 107.95) (xy 180.34 107.95))
     (stroke (width 0) (type default) (color 0 0 0 0))
@@
     (stroke (width 0) (type default) (color 0 0 0 0))
   )
-  (wire (pts (xy 33.02 16.51) (xy 33.02 19.05))
+  (wire (pts (xy 33.02 16.51) (xy 33.02 17.78))
     (stroke (width 0) (type default) (color 0 0 0 0))
   )
@@
     (stroke (width 0) (type default) (color 0 0 0 0))
   )
+  (wire (pts (xy 35.56 17.78) (xy 63.5 17.78))
+    (stroke (width 0) (type default) (color 0 0 0 0))
+  )
   (wire (pts (xy 116.84 41.91) (xy 116.84 44.45))
     (stroke (width 0) (type default) (color 0 0 0 0))
@@
     (stroke (width 0) (type default) (color 0 0 0 0))
   )
+  (wire (pts (xy 35.56 19.05) (xy 35.56 17.78))
+    (stroke (width 0) (type default) (color 0 0 0 0))
+  )
   (wire (pts (xy 60.96 39.37) (xy 60.96 38.1))
     (stroke (width 0) (type default) (color 0 0 0 0))
@@
     (stroke (width 0) (type default) (color 0 0 0 0))
   )
+  (wire (pts (xy 33.02 17.78) (xy 33.02 19.05))
+    (stroke (width 0) (type default) (color 0 0 0 0))
+  )
   (wire (pts (xy 152.4 106.68) (xy 152.4 107.95))
     (stroke (width 0) (type default) (color 0 0 0 0))
@@
   )
   (wire (pts (xy 168.91 142.24) (xy 168.91 168.91))
+    (stroke (width 0) (type default) (color 0 0 0 0))
+  )
+  (wire (pts (xy 63.5 17.78) (xy 63.5 19.05))
     (stroke (width 0) (type default) (color 0 0 0 0))
   )
@@
     (pin "9")
   )
+  (symbol (lib_id "Device:C") (at 63.5 22.86 180) (unit 1)
+    (in_bom yes) (on_board yes) (fields_autoplaced)
+    (property "Reference" "C19" (id 0) (at 67.31 21.5899 0)
+      (effects (font (size 1.27 1.27)) (justify right))
+    )
+    (property "Value" "100nF" (id 1) (at 67.31 24.1299 0)
+      (effects (font (size 1.27 1.27)) (justify right))
+    )
+    (property "Footprint" "Capacitor_SMD:C_0805_2012Metric" (id 2) (at 62.5348 19.05 0)
+      (effects (font (size 1.27 1.27)) hide)
+    )
+    (property "Datasheet" "~" (id 3) (at 63.5 22.86 0)
+      (effects (font (size 1.27 1.27)) hide)
+    )
+    (pin "1")
+    (pin "2")
+  )
   (symbol (lib_id "LED:NeoPixel_THT") (at 180.34 74.93 0) (unit 1)
     (in_bom yes) (on_board yes) (fields_autoplaced)
@@
     (pin "9")
   )
+  (symbol (lib_id "power:GND") (at 63.5 27.94 0) (unit 1)
+    (in_bom yes) (on_board yes) (fields_autoplaced)
+    (property "Reference" "#PWR010" (id 0) (at 63.5 34.29 0)
+      (effects (font (size 1.27 1.27)) hide)
+    )
+    (property "Value" "GND" (id 1) (at 63.5 33.02 0))
+    (property "Footprint" "" (id 2) (at 63.5 27.94 0)
+      (effects (font (size 1.27 1.27)) hide)
+    )
+    (property "Datasheet" "" (id 3) (at 63.5 27.94 0)
+      (effects (font (size 1.27 1.27)) hide)
+    )
+    (pin "1")
+  )
   (symbol (lib_id "Device:C") (at 158.75 180.34 0) (unit 1)
     (in_bom yes) (on_board yes)
@@
       (reference "#PWR09") (unit 1) (value "GND") (footprint "")
     )
+    (path "/cd08f49a-59f2-42e5-9af1-55696f36bce1"
+      (reference "#PWR010") (unit 1) (value "GND") (footprint "")
+    )
     (path "/6da1397b-dc7b-421c-ab0f-d00e0e6187a5"
       (reference "#PWR011") (unit 1) (value "GND") (footprint "")
@@
       (reference "C18") (unit 1) (value "22uF") (footprint "Capacitor_SMD:C_0805_2012Metric")
     )
+    (path "/82ef9c2f-7e78-4b18-89f3-7b2d4e4afabb"
+      (reference "C19") (unit 1) (value "100nF") (footprint "Capacitor_SMD:C_0805_2012Metric")
+    )
     (path "/8544b940-a52f-40fd-ae95-c83f0245f4b3"
