File: JF-Clock_template_rpi.kicad_pcb (KiCad board)
At the start: 2 copper layers, 177.7 x 56.2 mm, 75 parts, among them J1 Dh1, J10 Dm6, J11 USB_B_Micro, J12 Conn_01x02, J13 Conn_01x08_Female, J14 Conn_01x08_Female, J15 Conn_01x02, J2 Dh2, J3 Dh3, J4 Dh4, J5 Dm1, J6 Dm2, J7 Dm3, J8 Dm4, J9 Dm5, Q1 Q_PMOS_DSG, SW1 SW_Push, SW2 SW_Push, SW3 SW_Push, SW4 SW_Push, U1 MCP73831-2-OT, U2 TPS61200DRC, U4 DS3231M

Commit message: update for project
Parts:
- added D2: POWER LED, LED_SMD:LED_0603_1608Metric, F.Cu at (212.8, 129.3)
- added D3: CHARGE LED, LED_SMD:LED_0603_1608Metric, F.Cu at (211.1, 129.4)
- added JP1: SolderJumper_3_Bridged12, Jumper:SolderJumper-3_P1.3mm_Bridged12_RoundedPad1.0x1.5mm_NumberLabels, B.Cu at (157.2, 96.5)
- added JP3: PWR OUT, Jumper:SolderJumper-2_P1.3mm_Bridged_Pad1.0x1.5mm, F.Cu at (214.2, 123.0)
- added R5: 470, Resistor_SMD:R_0805_2012Metric, F.Cu at (214.0, 132.9)
- added R6: 1K, Resistor_SMD:R_0805_2012Metric, F.Cu at (210.2, 132.9)
- added TP2: 5V, TestPoint:TestPoint_THTPad_2.5x2.5mm_Drill1.2mm, F.Cu at (157.8, 89.2)
- added TP3: LEDPWR, TestPoint:TestPoint_THTPad_2.5x2.5mm_Drill1.2mm, F.Cu at (184.1, 86.4)
- added TP4: GND, TestPoint:TestPoint_THTPad_2.5x2.5mm_Drill1.2mm, F.Cu at (128.7, 82.5)
- A1: footprint Module:RaspberryPi_Pico_W_SMD_HandSolder -> Module:RaspberryPi_Pico_Common_THT
- moved VR1 62.4 mm to (99.6, 108.7)
- moved TP1 28.6 mm to (157.3, 82.5)
- moved TP7 27.7 mm to (128.9, 109.4)
- moved TP8 27.7 mm to (128.9, 113.5)
- moved J15 26.1 mm to (102.2, 120.8)
- moved A1 24.9 mm to (134.8, 83.0)
- moved R2 20.8 mm to (201.8, 120.7), turned to 90 degrees
- moved J14 18.0 mm to (124.0, 106.8)
- moved J13 18.0 mm to (106.0, 106.8)
- moved R8 17.9 mm to (110.5, 108.5), turned to 90 degrees
- moved R9 17.9 mm to (110.5, 112.0), turned to 90 degrees
- moved Q1 12.9 mm to (198.1, 123.3), turned to 0 degrees
- moved R7 9.87 mm to (177.8, 123.0)
- moved R1 8.72 mm to (192.3, 99.0), turned to 0 degrees
- moved R3 8.62 mm to (200.2, 133.4), turned to 0 degrees
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- renumbered J14 to J13, J13 to J14, JP1 to JP2, R8 to R10, R9 to R11, R5 to R7, R6 to R8, R7 to R9, TP2 to TP5, TP3 to TP6, TP4 to TP7, TP5 to TP8
Connections:
- A1 pad 36: unconnected-(A1-3V3-Pad36) -> /3v3
- C1 pad 1: /5v -> /Dh1_3
- C10 pad 1: /5v -> /Dh1_3
- C16 pad 1: /5v -> Net-(D1-K)
- C2 pad 1: /5v -> /Dh1_3
- C3 pad 1: /5v -> /Dh1_3
- C4 pad 1: /5v -> /Dh1_3
- C5 pad 1: /5v -> /Dh1_3
- C6 pad 1: /5v -> /Dh1_3
- C7 pad 1: /5v -> /Dh1_3
- C8 pad 1: /5v -> /Dh1_3
- C9 pad 1: /5v -> /Dh1_3
- D1 pad 1: /5v -> Net-(D1-K)
- Dh1 pad 3: /5v -> /Dh1_3
- Dh2 pad 3: /5v -> /Dh1_3
- Dh3 pad 3: /5v -> /Dh1_3
- Dh4 pad 3: /5v -> /Dh1_3
- Dm1 pad 3: /5v -> /Dh1_3
- Dm2 pad 3: /5v -> /Dh1_3
- Dm3 pad 3: /5v -> /Dh1_3
- Dm4 pad 3: /5v -> /Dh1_3
- Dm5 pad 3: /5v -> /Dh1_3
- Dm6 pad 3: /5v -> /Dh1_3
- J1 pad 3: /5v -> /Dh1_3
- J10 pad 3: /5v -> /Dh1_3
- J2 pad 3: /5v -> /Dh1_3
- J3 pad 3: /5v -> /Dh1_3
- J4 pad 3: /5v -> /Dh1_3
- J5 pad 3: /5v -> /Dh1_3
- J6 pad 3: /5v -> /Dh1_3
- J7 pad 3: /5v -> /Dh1_3
- J8 pad 3: /5v -> /Dh1_3
- J9 pad 3: /5v -> /Dh1_3
- U1 pad 1: unconnected-(U1-STAT-Pad1) -> Net-(U1-STAT)
- U2 pad 10: /5v -> Net-(D1-K)
- U2 pad 2: /5v -> Net-(D1-K)
- VR1 pad 1: /5v -> /3v3
Routing:
- net /5v: track 595.9 -> 217.6 mm, vias 2 -> 3
- net /Dh1_3: track 0.00 -> 324.4 mm, vias 0 -> 10
- net /3v3: track 0.00 -> 69.0 mm
- net GND: track 159.8 -> 91.5 mm, vias 32 -> 6
- net Net-(D1-K): track 0.00 -> 65.9 mm, vias 0 -> 2
- net Net-(BT2-+): track 33.7 -> 63.2 mm
- net /NeoPixel_D: track 53.8 -> 83.2 mm
- net Net-(Q1-D): track 75.4 -> 51.9 mm
- net Net-(A1-VBUS): track 25.9 -> 4.96 mm
- net Net-(D1-A): track 62.0 -> 42.9 mm
- net /Dm2_Out: track 61.8 -> 50.2 mm
- net Net-(U1-STAT): track 0.00 -> 11.6 mm
- net /Dh1_In: track 27.5 -> 16.5 mm, vias 1 -> 0
- net /Dh4_Out: track 115.0 -> 104.4 mm, vias 2 -> 0
- net /Dm5_Out: track 54.7 -> 44.2 mm
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- added copper zone on F.Cu, net GND
Other:
- board text added: "CHARGE LED"
- board text added: "JOEY FRANK CLOCK TEMPLATE JPC003 REV2"
- board text added: "POWER LED"
- board text removed: "JOEY FRANK CLOCK TEMPLATE JPC003"
