File: JF-Clock_template_rpi.kicad_sch (KiCad schematic)
At the start: 73 parts, among them J1 Dh1, J10 Dm6, J11 USB_B_Micro, J12 Conn_01x02, J13 Conn_01x08_Female, J14 Conn_01x08_Female, J15 Conn_01x02, J2 Dh2, J3 Dh3, J4 Dh4, J5 Dm1, J6 Dm2, J7 Dm3, J8 Dm4, J9 Dm5, Q1 Q_PMOS_DSG, SW1 SW_Push, SW2 SW_Push, SW3 SW_Push, SW4 SW_Push, U1 MCP73831-2-OT, U2 TPS61200DRC, U3 DFR0299, U4 DS3231M

Commit message: update for project
Parts:
- added D2: POWER LED, LED_SMD:LED_0603_1608Metric, symbol Device:LED
- added D3: CHARGE LED, LED_SMD:LED_0603_1608Metric, symbol Device:LED
- added JP1: SolderJumper_3_Bridged12, Jumper:SolderJumper-3_P1.3mm_Bridged12_RoundedPad1.0x1.5mm_NumberLabels, symbol Jumper:SolderJumper_3_Bridged12
- added JP3: PWR OUT, Jumper:SolderJumper-2_P1.3mm_Bridged_Pad1.0x1.5mm, symbol Jumper:SolderJumper_2_Bridged
- added R5: 470, Resistor_SMD:R_0805_2012Metric, symbol Device:R
- added R6: 1K, Resistor_SMD:R_0805_2012Metric, symbol Device:R
- added TP2: 5V, TestPoint:TestPoint_THTPad_2.5x2.5mm_Drill1.2mm, symbol Connector:TestPoint
- added TP3: LEDPWR, TestPoint:TestPoint_THTPad_2.5x2.5mm_Drill1.2mm, symbol Connector:TestPoint
- added TP4: GND, TestPoint:TestPoint_THTPad_2.5x2.5mm_Drill1.2mm, symbol Connector:TestPoint
- A1: footprint Module:RaspberryPi_Pico_W_SMD_HandSolder -> Module:RaspberryPi_Pico_Common_THT
- LS1: footprint (none) -> TestPoint:TestPoint_Bridge_Pitch2.54mm_Drill1.0mm
- renumbered J14 to J13, J13 to J14, JP1 to JP2, R8 to R10, R9 to R11, R5 to R7, R6 to R8, R7 to R9, TP2 to TP5, TP3 to TP6, TP4 to TP7, TP5 to TP8
Connections:
- net 5v: now also D2.2 (A), JP1.3 (B), JP3.2 (B), TP2.1; no longer C1.1, C10.1, C16.1, C2.1, C3.1, C4.1, C5.1, C6.1, C7.1, C8.1, C9.1, D1.1 (K), Dh1.3 (VDD), Dh2.3 (VDD), Dh3.3 (VDD), Dh4.3 (VDD), Dm1.3 (VDD), Dm2.3 (VDD), Dm3.3 (VDD), Dm4.3 (VDD), Dm5.3 (VDD), Dm6.3 (VDD), J1.3 (Pin_3), J10.3 (Pin_3), J2.3 (Pin_3), J3.3 (Pin_3), J4.3 (Pin_3), J5.3 (Pin_3), J6.3 (Pin_3), J7.3 (Pin_3), J8.3 (Pin_3), J9.3 (Pin_3), U2.10 (FB), U2.2 (VOUT), VR1.1
- net GND: now also R5.1, TP4.1
- net at U1.1 (STAT): now also R6.1
- net 3v3: now reaches A1.36 (3V3)
- net 3v3: now also VR1.1, JP1.1 (A)
- new net: D2.1 (K), R5.2
- new net: D3.1 (K), R6.2
- new net: C16.1, D1.1 (K), JP3.1 (A), U2.10 (FB), U2.2 (VOUT)
- new net Dh1_3: C1.1, C10.1, C2.1, C3.1, C4.1, C5.1, C6.1, C7.1, C8.1, C9.1, Dh1.3 (VDD), Dh2.3 (VDD), Dh3.3 (VDD), Dh4.3 (VDD), Dm1.3 (VDD), Dm2.3 (VDD), Dm3.3 (VDD), Dm4.3 (VDD), Dm5.3 (VDD), Dm6.3 (VDD), J1.3 (Pin_3), J10.3 (Pin_3), J2.3 (Pin_3), J3.3 (Pin_3), J4.3 (Pin_3), J5.3 (Pin_3), J6.3 (Pin_3), J7.3 (Pin_3), J8.3 (Pin_3), J9.3 (Pin_3), JP1.2 (C), TP3.1
- new net VDD: D3.2 (A)
- no-connect marks 49 -> 47
Other:
- note added: "TODO: - Change dimmer to knob/slider that is also the power, bonus is a slider that triggers a pitchslide sound - Audio tester button, if pressed twice increments to next set sound in list - fix debounce to be more responsive, if we cant fix it then change buttons - new switch for swapping reading direction, with indicator Bonus: - test circuit of capacitive touch slider - test circuit of diffuse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"
- note removed: "TODO: - Change dimmer to knob/slider that is also the power, bonus is a slider that triggers a pitchslide sound - Audio tester button, if pressed twice increments to next set sound in list - fix debounce to be more responsive, if we cant fix it then change buttons - new switch for swapping reading direction, with indicator - blue wire mistake! Bonus: - test circuit of capacitive touch slider - te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"
- moved on the sheet: C12, J13, J14, J15, LS1, R8, R9, TP1, TP7, TP8
